File: light sensor basic.brd (EAGLE design)
At the start: 83.2 x 57.8 mm, 1 part

Commit message: eagle assignment 2
Parts:
- added C1: 0.1 uF, rcl:C1206
- added J1: UJ2-MIBH-G-SMT-TR, UJ2-MIBH-G-SMT-TR:CUI_UJ2-MIBH-G-SMT-TR
- added LED1: (no value), led:SML0805
- added R1: (no value), rcl:R0805
- added R2: TC33X-2-203E, TC33X-2-203E:TRIM_TC33X-2-203E
- added R3: 150, rcl:R0805
- added T1: (no value), transistor-neu-to92:SOT23-BEC
- added TP1, TP2, TP3, TP4: (no value), rcl:R1206
- added U1: VCNT2020, VCNT2020:XDCR_VCNT2020
Connections:
- new net GND: C1.1, J1.5, J1.S1, J1.S2, J1.S3, J1.S4, R2.3, T1.E, TP4.1, TP4.2, U1.4
- new net N$1: R1.1, U1.3
- new net N$2: R2.1, TP1.1, TP1.2, U1.1
- new net N$3: R2.2, T1.B, TP2.1, TP2.2
- new net N$4: LED1.C, T1.C
- new net N$5: LED1.A, R3.1
- new net VCC: C1.2, J1.1, R1.2, R3.2, TP3.1, TP3.2, U1.2
